File: Power_suppy.sch (KiCad schematic (older format))
At the start: 12 parts, among them J3 Conn_01x02_Female, U3 LM2596S-5, U4 LM1117-3.3

Commit message: reorganized schematic; added reverse polarity protection; start adding footprints
Parts:
- C11: value C_Small -> 1uF
- C12: value CP_Small -> 100uF
- C13, C14: value C_Small -> 100nF
- C15: value CP_Small -> 220uF
- L2: value L_Small -> 33uH
Connections:
- wire segments 40 -> 47
Other:
- moved on the sheet: C11, C12, C13, C14, C15, D2
Changed lines of the file:
@@
 $Descr A4 11693 8268
 encoding utf-8
-Sheet 3 7
+Sheet 3 10
 Title "PUTM_EV_Dashboard_2021"
 Date ""
@@
 L Connector:Conn_01x02_Female J3
 U 1 1 61C14982
-P 3200 2450
-F 0 "J3" H 3094 2125 50  0000 C CNN
-F 1 "Conn_01x02_Female" H 3094 2216 50  0000 C CNN
-F 2 "" H 3200 2450 50  0001 C CNN
-F 3 "~" H 3200 2450 50  0001 C CNN
-	1    3200 2450
+P 2800 2450
+F 0 "J3" H 2694 2125 50  0000 C CNN
+F 1 "Conn_01x02_Female" H 2694 2216 50  0000 C CNN
+F 2 "" H 2800 2450 50  0001 C CNN
+F 3 "~" H 2800 2450 50  0001 C CNN
+	1    2800 2450
 	-1   0    0    1
 $EndComp
@@
 	3500 2500 3500 2450
 Wire Wire Line
-	3500 2450 3400 2450
+	3500 2450 3000 2450
 $Comp
 L Device:Fuse F1
@@
 $EndComp
 Wire Wire Line
-	3550 2350 3400 2350
-Wire Wire Line
-	3850 2350 3950 2350
+	3550 2350 3000 2350
 $Comp
 L Device:D_Schottky D2
 U 1 1 61C14CE8
-P 3950 2500
-F 0 "D2" V 3904 2579 50  0000 L CNN
-F 1 "D_Schottky" V 3995 2579 50  0000 L CNN
-F 2 "" H 3950 2500 50  0001 C CNN
-F 3 "~" H 3950 2500 50  0001 C CNN
-	1    3950 2500
+P 3950 2650
+F 0 "D2" V 3904 2729 50  0000 L CNN
+F 1 "D_Schottky" V 3995 2729 50  0000 L CNN
+F 2 "" H 3950 2650 50  0001 C CNN
+F 3 "~" H 3950 2650 50  0001 C CNN
+	1    3950 2650
 	0    1    1    0
 $EndComp
-Connection ~ 3950 2350
-Wire Wire Line
-	3950 2350 4250 2350
 $Comp
 L Device:C_Small C11
 U 1 1 61C14D81
-P 4250 2450
-F 0 "C11" H 4342 2496 50  0000 L CNN
-F 1 "C_Small" H 4342 2405 50  0000 L CNN
-F 2 "" H 4250 2450 50  0001 C CNN
-F 3 "~" H 4250 2450 50  0001 C CNN
-	1    4250 2450
-	1    0    0    -1
-$EndComp
-Connection ~ 4250 2350
-Wire Wire Line
-	4250 2350 4550 2350
+P 7350 2750
+F 0 "C11" H 7442 2796 50  0000 L CNN
+F 1 "1uF" H 7442 2705 50  0000 L CNN
+F 2 "" H 7350 2750 50  0001 C CNN
+F 3 "~" H 7350 2750 50  0001 C CNN
+	1    7350 2750
+	1    0    0    -1
+$EndComp
 $Comp
 L Device:CP_Small C12
 U 1 1 61C14E07
-P 4550 2450
-F 0 "C12" H 4638 2496 50  0000 L CNN
-F 1 "CP_Small" H 4638 2405 50  0000 L CNN
-F 2 "" H 4550 2450 50  0001 C CNN
-F 3 "~" H 4550 2450 50  0001 C CNN
-	1    4550 2450
-	1    0    0    -1
-$EndComp
-Connection ~ 4550 2350
-Wire Wire Line
-	4550 2350 4900 2350
+P 4550 2600
+F 0 "C12" H 4650 2600 50  0000 L CNN
+F 1 "100uF" H 4550 2500 50  0000 L CNN
+F 2 "" H 4550 2600 50  0001 C CNN
+F 3 "~" H 4550 2600 50  0001 C CNN
+	1    4550 2600
+	1    0    0    -1
+$EndComp
 $Comp
 L power:GND #PWR0124
@@
 Wire Wire Line
 	5400 2950 4800 2950
-Wire Wire Line
-	3950 2950 3950 2650
 Connection ~ 5400 2950
-Wire Wire Line
-	4250 2550 4250 2950
-Connection ~ 4250 2950
-Wire Wire Line
-	4250 2950 3950 2950
-Wire Wire Line
-	4550 2550 4550 2950
-Connection ~ 4550 2950
-Wire Wire Line
-	4550 2950 4250 2950
 Wire Wire Line
 	4900 2550 4800 2550
@@
 	4800 2550 4800 2950
 Connection ~ 4800 2950
-Wire Wire Line
-	4800 2950 4550 2950
 $Comp
 L Device:D_Schottky D3
@@
 U 1 1 61C1556A
 P 6450 2550
-F 0 "L2" V 6635 2550 50  0000 C CNN
-F 1 "L_Small" V 6544 2550 50  0000 C CNN
+F 0 "L2" V 6400 2450 50  0000 C CNN
+F 1 "33uH" V 6544 2550 50  0000 C CNN
 F 2 "" H 6450 2550 50  0001 C CNN
 F 3 "~" H 6450 2550 50  0001 C CNN
@@
 L Device:CP_Small C15
 U 1 1 61C155DD
-P 6950 2650
-F 0 "C15" H 7038 2696 50  0000 L CNN
-F 1 "CP_Small" H 7038 2605 50  0000 L CNN
-F 2 "" H 6950 2650 50  0001 C CNN
-F 3 "~" H 6950 2650 50  0001 C CNN
-	1    6950 2650
+P 6950 2750
+F 0 "C15" H 7038 2796 50  0000 L CNN
+F 1 "220uF" H 7038 2705 50  0000 L CNN
+F 2 "" H 6950 2750 50  0001 C CNN
+F 3 "~" H 6950 2750 50  0001 C CNN
+	1    6950 2750
 	1    0    0    -1
 $EndComp
@@
 Connection ~ 6950 2550
 Wire Wire Line
-	6950 2750 6950 2950
-Wire Wire Line
 	6950 2950 6200 2950
 Wire Wire Line
@@
 	6200 2950 5400 2950
 Wire Wire Line
-	6950 2550 7600 2550
+	6950 2550 7350 2550
 Wire Wire Line
 	7600 2550 7600 2450
@@
 L Device:C_Small C13
 U 1 1 61C1689F
-P 4800 3900
-F 0 "C13" H 4892 3946 50  0000 L CNN
-F 1 "C_Small" H 4892 3855 50  0000 L CNN
-F 2 "" H 4800 3900 50  0001 C CNN
-F 3 "~" H 4800 3900 50  0001 C CNN
-	1    4800 3900
+P 4800 3950
+F 0 "C13" H 4892 3996 50  0000 L CNN
+F 1 "100nF" H 4892 3905 50  0000 L CNN
+F 2 "" H 4800 3950 50  0001 C CNN
+F 3 "~" H 4800 3950 50  0001 C CNN
+	1    4800 3950
 	1    0    0    -1
 $EndComp
@@
 L Device:C_Small C14
 U 1 1 61C1691D
-P 6200 3900
-F 0 "C14" H 6292 3946 50  0000 L CNN
-F 1 "C_Small" H 6292 3855 50  0000 L CNN
-F 2 "" H 6200 3900 50  0001 C CNN
-F 3 "~" H 6200 3900 50  0001 C CNN
-	1    6200 3900
+P 6000 3950
+F 0 "C14" H 6092 3996 50  0000 L CNN
+F 1 "100nF" H 6092 3905 50  0000 L CNN
+F 2 "" H 6000 3950 50  0001 C CNN
+F 3 "~" H 6000 3950 50  0001 C CNN
+	1    6000 3950
 	1    0    0    -1
 $EndComp
@@
 $EndComp
 Wire Wire Line
-	5450 4250 5450 4100
-Wire Wire Line
-	5450 4100 4800 4100
-Wire Wire Line
-	4800 4100 4800 4000
-Connection ~ 5450 4100
-Wire Wire Line
-	4800 3800 5150 3800
-Wire Wire Line
 	4650 3550 4650 3800
-Wire Wire Line
-	4650 3800 4800 3800
-Connection ~ 4800 3800
-Wire Wire Line
-	6200 3800 5750 3800
-Wire Wire Line
-	6200 4000 6200 4100
-Wire Wire Line
-	6200 4100 5450 4100
 $Comp
 L power:+3.3V #PWR0128
 U 1 1 61C17EDA
-P 6850 3600
-F 0 "#PWR0128" H 6850 3450 50  0001 C CNN
-F 1 "+3.3V" H 6865 3773 50  0000 C CNN
-F 2 "" H 6850 3600 50  0001 C CNN
-F 3 "" H 6850 3600 50  0001 C CNN
-	1    6850 3600
-	1    0    0    -1
-$EndComp
-Wire Wire Line
-	6850 3600 6850 3800
-Wire Wire Line
-	6850 3800 6200 3800
-Connection ~ 6200 3800
+P 6400 3600
+F 0 "#PWR0128" H 6400 3450 50  0001 C CNN
+F 1 "+3.3V" H 6415 3773 50  0000 C CNN
+F 2 "" H 6400 3600 50  0001 C CNN
+F 3 "" H 6400 3600 50  0001 C CNN
+	1    6400 3600
+	1    0    0    -1
+$EndComp
+Wire Wire Line
+	6400 3600 6400 3800
 Wire Wire Line
 	6200 2600 6200 2550
@@
 Wire Wire Line
 	6200 2550 6350 2550
+Wire Wire Line
+	6950 2550 6950 2650
+Wire Wire Line
+	6950 2850 6950 2950
+Wire Wire Line
+	3850 2350 3950 2350
+Wire Wire Line
+	3950 2950 4550 2950
+Wire Wire Line
+	4550 2950 4550 2700
+Connection ~ 4550 2950
+Wire Wire Line
+	4550 2950 4800 2950
+Connection ~ 4550 2350
+Wire Wire Line
+	4550 2350 4900 2350
+Wire Wire Line
+	4550 2500 4550 2350
+Wire Wire Line
+	6950 2950 7350 2950
+Wire Wire Line
+	7350 2950 7350 2850
+Connection ~ 6950 2950
+Wire Wire Line
+	7350 2650 7350 2550
+Connection ~ 7350 2550
+Wire Wire Line
+	7350 2550 7600 2550
+Wire Wire Line
+	3950 2500 3950 2350
+Connection ~ 3950 2350
+Wire Wire Line
+	3950 2350 4550 2350
+Wire Wire Line
+	3950 2800 3950 2950
+Wire Wire Line
+	4800 4150 5450 4150
+Wire Wire Line
+	4650 3800 4800 3800
+Wire Wire Line
+	5750 3800 6000 3800
+Wire Wire Line
+	6000 3800 6000 3850
+Connection ~ 6000 3800
+Wire Wire Line
+	6000 3800 6400 3800
+Wire Wire Line
+	6000 4050 6000 4150
+Wire Wire Line
+	5450 4100 5450 4150
+Connection ~ 5450 4150
+Wire Wire Line
+	5450 4150 6000 4150
+Wire Wire Line
+	5450 4150 5450 4250
+Wire Wire Line
+	4800 4150 4800 4050
+Connection ~ 4800 3800
+Wire Wire Line
+	4800 3800 5150 3800
+Wire Wire Line
+	4800 3850 4800 3800
 $EndSCHEMATC
