File: dash_hw.kicad_pcb (KiCad board)
At the start: 2 copper layers, 195 parts, among them J1 Conn_01x04, J2 USB_B_Mini, J3 Conn_01x06_Male, Q1 DMP3056L-7, SW1 SW_Push, U1 LM1117-3.3, U10 FT232RL, U11 74HC595, U12 74HC595, U13 74HC595, U14 74HC595, U17 74HC595, U19 74HC595, U2 LM2596S-5, U20 STM32F103C8Tx, U3 MCP2562-H-SN, U4 74HC595, U5 74HC595, U6 74HC595, U7 OPS-S5621, U8 OPS-S5621, U9 OPS-S5621, Y1 Crystal

Commit message: remove double elements in 3state leds
Parts:
- removed D49, D50, D51, D52, D53, D54: LED, LED_THT:LED_D3.0mm_Clear
- removed R75, R76, R77, R78, R79, R80: 200, Resistor_SMD:R_0603_1608Metric
- C14, D79, D80, D81, D82, R105, R106, R107, R108, R109, RV1, SW1: moved to B.Cu
- U12, U13: moved to F.Cu
- moved C17 349.6 mm to (270.1, 141.5)
- moved C18 349.6 mm to (280.4, 131.3)
- moved C19 349.6 mm to (270.1, 139.0)
- moved C21 349.6 mm to (266.1, 141.5)
- moved J3 349.6 mm to (250.4, 127.3)
- moved L3 349.6 mm to (278.2, 133.8)
- moved C20 339.1 mm to (264.3, 132.1)
- moved D41 337.9 mm to (223.5, 95.2)
- moved D48 333.6 mm to (234.9, 114.3)
- moved U17 331.1 mm to (208.3, 106.7)
- moved D44 327.3 mm to (224.8, 105.4)
- moved D42 323.5 mm to (231.1, 95.2)
- moved D40 318.8 mm to (214.6, 95.2)
- moved D45 316.5 mm to (233.7, 105.4)
- moved C14 316.0 mm to (230.7, 131.4)
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Other:
- board outline added: 180.3 x 73.7 mm

Commit message: Hardware update Approved
Parts:
- removed D10, D11, D12, D13, D14, D7, D8, D9: LED, LED_THT:LED_D3.0mm_Clear
- removed R33, R34, R35, R36, R37, R38, R39, R40: 200, Resistor_SMD:R_0603_1608Metric
- removed U11: 74HC595, Package_SO:SOIC-16_3.9x9.9mm_P1.27mm
- added C22: 470nF, Capacitor_SMD:C_1206_3216Metric, B.Cu at (71.8, 76.0)
- added D49: LED_Small, LED_THT:LED_D3.0mm_Clear, F.Cu at (63.6, 89.2)
- added D50: LED_Small, LED_THT:LED_D3.0mm_Clear, F.Cu at (72.6, 89.2)
- added D51: LED_Small, LED_THT:LED_D3.0mm_Clear, F.Cu at (81.6, 89.2)
- added D52: LED_Small, LED_THT:LED_D3.0mm_Clear, F.Cu at (188.6, 89.2)
- added D53: LED_Small, LED_THT:LED_D3.0mm_Clear, F.Cu at (197.6, 89.1)
- added D54: LED_Small, LED_THT:LED_D3.0mm_Clear, F.Cu at (206.6, 89.1)
- added F2: Polyfuse, Fuse:Fuse_2010_5025Metric, B.Cu at (113.5, 94.2)
- added J4: Conn_01x06_Female, Connector_PinHeader_2.54mm:PinHeader_1x06_P2.54mm_Vertical, F.Cu at (62.4, 112.4)
- added R75: 200R, Capacitor_SMD:C_0603_1608Metric, B.Cu at (64.7, 95.2)
- added R76: 200R, Capacitor_SMD:C_0603_1608Metric, B.Cu at (73.9, 94.4)
- added R77: 200R, Capacitor_SMD:C_0603_1608Metric, B.Cu at (82.6, 94.8)
- added R78: 200R, Capacitor_SMD:C_0603_1608Metric, B.Cu at (189.9, 93.9)
- added R79: 200R, Capacitor_SMD:C_0603_1608Metric, B.Cu at (199.0, 94.0)
- added R80: 200R, Capacitor_SMD:C_0603_1608Metric, B.Cu at (207.6, 93.8)
- added R81: R_Small, Capacitor_SMD:C_0603_1608Metric, B.Cu at (64.7, 92.9)
- added R82: R_Small, Capacitor_SMD:C_0603_1608Metric, B.Cu at (74.0, 92.5)
- added R83: R_Small, Capacitor_SMD:C_0603_1608Metric, B.Cu at (82.6, 92.6)
- added R84: R_Small, Capacitor_SMD:C_0603_1608Metric, B.Cu at (189.7, 92.1)
- added R85: R_Small, Capacitor_SMD:C_0603_1608Metric, B.Cu at (199.0, 92.1)
- added R86: R_Small, Capacitor_SMD:C_0603_1608Metric, B.Cu at (207.7, 92.1)
- C1, C10, C11, C12, C13, C15, C16, C17, C18, C19, C2, C20, C21, C4, C6, C7, C8, C9, D1, D2, D3, D4, D5, D6, F1, J2, J3, JP1, L1, L3, Q1, R1, R110, R2, R27, R28, R31, U1, U10, U19, U2, U20, U3, Y1: moved to B.Cu
- C3, C5: footprint Capacitor_SMD:CP_Elec_8x10 -> Capacitor_THT:CP_Radial_D6.3mm_P2.50mm; moved to B.Cu
- L2: value L -> KoralikFerrytowy; moved to B.Cu
- R29, R30: value 1k -> 560R; moved to B.Cu
- R32: value R -> 0R
- RV1: value R_POT -> 10k
- U7, U8, U9: footprint PUTM_EV_Dashboard_2021:OPS-S5621LB-GW -> PUTMotorsport_footprints:0.56” Case Mold Type LED Display
- moved U19 323.5 mm to (195.8, 135.4), turned to 270 degrees
- moved R69 302.4 mm to (189.9, 117.5), turned to 180 degrees
- moved R68 298.2 mm to (201.9, 105.3), turned to 180 degrees
- moved R74 295.2 mm to (201.9, 129.5), turned to 180 degrees
- moved R71 294.6 mm to (201.9, 117.5), turned to 180 degrees
- moved R66 286.2 mm to (189.9, 105.3), turned to 180 degrees
- moved R70 283.4 mm to (196.0, 117.5), turned to 180 degrees
- moved R72 279.7 mm to (189.9, 129.5), turned to 180 degrees
- moved R67 278.5 mm to (196.0, 105.3), turned to 180 degrees
- moved R73 276.7 mm to (195.8, 129.5), turned to 180 degrees
- moved J2 273.2 mm to (207.7, 78.9), turned to 270 degrees
- moved L2 263.8 mm to (200.3, 76.4), turned to 90 degrees
- moved C9 257.7 mm to (202.1, 76.4), turned to 270 degrees
- moved D6 256.7 mm to (186.4, 85.0), turned to 90 degrees
- moved D5 254.5 mm to (188.1, 85.0), turned to 90 degrees
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Connections:
- J1 pad 3: /CAN- -> /CANL
Routing:
- net +5V: track 0.00 -> 564.1 mm, vias 0 -> 23
- net +3V3: track 0.00 -> 345.4 mm, vias 0 -> 11
- net /SPI_2_CS: track 0.00 -> 285.4 mm, vias 0 -> 3
- net /SPI_2_CLK: track 0.00 -> 264.0 mm, vias 0 -> 6
- net /CANL: track 0.00 -> 201.6 mm, vias 0 -> 4
- net /CANH: track 0.00 -> 198.5 mm, vias 0 -> 6
- net GND: track 0.00 -> 180.5 mm, vias 0 -> 58
- net FAULT1: track 0.00 -> 163.2 mm, vias 0 -> 1
- net 5Vfused: track 0.00 -> 160.4 mm, vias 0 -> 4
- net FAULT2: track 0.00 -> 156.2 mm, vias 0 -> 1
- net Net-(R65-Pad2): track 0.00 -> 152.7 mm
- net FAULT3: track 0.00 -> 148.5 mm, vias 0 -> 1
- net Net-(U14-Pad9): track 0.00 -> 116.6 mm, vias 0 -> 4
- net /mcu/LCD_RS: track 0.00 -> 100.7 mm, vias 0 -> 1
- net /display_16x2/E: track 0.00 -> 93.9 mm, vias 0 -> 1
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- added copper zone on B.Cu, net GND
- added copper zone on F.Cu, net GND
Other:
- board size 180.3 x 73.7 mm -> 155 x 70 mm
- net class 0.3 added: clearance 0.2, trace_width 0.35, via_dia 0.8, via_drill 0.4
- net class 0.8 added: clearance 0.2, trace_width 0.8, via_dia 0.8, via_drill 0.4
- net class 5v added: clearance 0.2, trace_width 0.5, via_dia 0.8, via_drill 0.4
- net class Zasilanie added: clearance 0.2, trace_width 1, via_dia 0.8, via_drill 0.4
- board text added: "LINIOWA:"
- board text added: "TOLERANCJE:"

Commit message: Updated hardware
Parts:
- removed J1: Conn_01x04, Connector_PinHeader_2.54mm:PinHeader_1x04_P2.54mm_Vertical
- added J5: Conn_01x02, Connector_PinHeader_2.54mm:PinHeader_1x02_P2.54mm_Vertical, F.Cu at (62.4, 104.6)
- added J6: Conn_01x02, Connector_PinHeader_2.54mm:PinHeader_1x02_P2.54mm_Vertical, F.Cu at (212.0, 111.6)
- moved JP1 3.82 mm to (196.6, 110.7), turned to 90 degrees
- moved R2 1.61 mm to (196.5, 108.2), turned to 180 degrees
- moved C6 1.55 mm to (106.6, 95.9), turned to 90 degrees
- moved C11 0.31 mm to (188.2, 72.8)
- turned D4 to 180 degrees
Routing:
- net /CANL: track 201.6 -> 20.9 mm, vias 4 -> 0
- net /CANH: track 198.5 -> 20.8 mm, vias 6 -> 0
- net GND: track 180.5 -> 189.9 mm, vias 58 -> 118
- net +5V: track 564.1 -> 558.1 mm
- net /GLV+: track 18.1 -> 21.7 mm
- net /SPI_2_CLK: track 264.0 -> 267.5 mm
- net Net-(D3-Pad1): track 32.6 -> 29.4 mm
- net /mcu/SW_NRST: track 57.1 -> 54.6 mm
- net FAULT3: track 148.5 -> 146.1 mm
- net /UART_RTS: track 29.3 -> 27.5 mm
- net /UART_CTS: track 24.9 -> 23.4 mm
- net FAULT2: track 156.2 -> 155.2 mm
- net /UART_RX: track 23.9 -> 23.1 mm
- net /display_16x2/D7: track 66.6 -> 65.8 mm
- net +3V3: track 345.4 -> 346.2 mm
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Other:
- board text removed: "LINIOWA:"
- board text removed: "TOLERANCJE:"
